Commit message: fix: floor friction and collisions

File: discower_cosmo/urdf/model.urdf (robot description, URDF)
Before this commit: robot discower_cosmo, 1 links, 0 joints
Links:
- link body: geometry collision box size=0.63 0.04 0.04; collision box size=0.78 0.04 0.04

File: discower_description/urdf/model.urdf.xacro (robot description, xacro)
@@ -31,5 +31,5 @@
     <self_collide>false</self_collide>
     <!-- body -->
-    <visual name="body_visual">
+    <visual>
       <origin xyz="0 0 0" rpy="0 0 0" />
       <geometry>
@@ -37,5 +37,5 @@
       </geometry>
     </visual>
-    <collision name="body_collision">
+    <collision>
       <origin xyz="0 0 0.25" rpy="0 0 0" />
       <geometry>
@@ -58,4 +58,11 @@
     <child link="${prefix}inertial_link" />
   </joint>
+  <gazebo reference="${prefix}body">
+    <kp>100000.0</kp>
+    <kd>100000.0</kd>
+    <mu1>0.0</mu1>
+    <mu2>0.</mu2>
+    <fdir1>0 0 1</fdir1>
+  </gazebo>
   <!-- MODEL-->
   <xacro:include filename="$(find discower_description)/urdf/model_drag.urdf.xacro" />
