Commit message: feat: adding thruster for gazebo

File: discower_description/urdf/model.urdf.xacro (robot description, xacro)
@@ -18,15 +18,9 @@
 <robot name="orion" xmlns:xacro="http://www.ros.org/wiki/xacro">
   <!-- OPTIONS -->
-  <xacro:property name="world" value="$(arg world)"/>
-  <xacro:property name="pay_top_aft" value="$(arg top_aft)"/>
-  <xacro:property name="pay_bot_aft" value="$(arg bot_aft)"/>
-  <xacro:property name="pay_bot_front" value="$(arg bot_front)"/>
-  <xacro:property name="ns" value="$(arg ns)"/>
   <xacro:property name="prefix" value="$(arg prefix)"/>
   <xacro:if value="${prefix == '/'}">
     <xacro:property name="prefix" value=""/>
   </xacro:if>
-  <!-- BASE GEOMETRY -->
- <link name="${prefix}body">
+  <link name="${prefix}body">
     <self_collide>false</self_collide>
     <!-- body -->
@@ -58,4 +52,133 @@
     <child link="${prefix}inertial_link" />
   </joint>
+  <!-- Thrusters links and joints-->
+  <link name="${prefix}thruster_0">
+    <self_collide>false</self_collide>
+    <inertial>
+      <mass value="0.001"/>
+      <origin xyz="-0.12 0.12 0.2" rpy="0 1.5708 0"/>
+      <inertia ixx="0.00001" ixy="0.0" ixz="0.0" iyy="0.00001" iyz="0.0" izz="0.00001"/>
+    </inertial>
+  </link>
+  <joint name='${prefix}thruster_0_joint' type='fixed'>
+    <parent link="${prefix}body" />
+    <child link="${prefix}thruster_0" />
+    <use_parent_model_frame>1</use_parent_model_frame>
+  </joint>
+  <gazebo reference="${prefix}thruster_0_joint">
+    <preserveFixedJoint>true</preserveFixedJoint>
+  </gazebo>
+  <link name="${prefix}thruster_1">
+    <self_collide>false</self_collide>
+    <inertial>
+      <mass value="0.001"/>
+      <origin xyz="0.12 0.12 0.2" rpy="0 -1.5708 0"/>
+      <inertia ixx="0.00001" ixy="0.0" ixz="0.0" iyy="0.00001" iyz="0.0" izz="0.00001"/>
+    </inertial>
+  </link>
+  <joint name='${prefix}thruster_1_joint' type='fixed'>
+    <parent link="${prefix}body" />
+    <child link="${prefix}thruster_1" />
+    <use_parent_model_frame>1</use_parent_model_frame>
+  </joint>
+  <gazebo reference="${prefix}thruster_1_joint">
+    <preserveFixedJoint>true</preserveFixedJoint>
+  </gazebo>
+  <link name="${prefix}thruster_2">
+    <self_collide>false</self_collide>
+    <inertial>
+      <mass value="0.001"/>
+      <origin xyz="-0.12 -0.12 0.2" rpy="0 1.5708 0"/>
+      <inertia ixx="0.00001" ixy="0.0" ixz="0.0" iyy="0.00001" iyz="0.0" izz="0.00001"/>
+    </inertial>
+  </link>
+  <joint name='${prefix}thruster_2_joint' type='fixed'>
+    <parent link="${prefix}body" />
+    <child link="${prefix}thruster_2" />
+    <use_parent_model_frame>1</use_parent_model_frame>
+  </joint>
+  <gazebo reference="${prefix}thruster_2_joint">
+    <preserveFixedJoint>true</preserveFixedJoint>
+  </gazebo>
+  <link name="${prefix}thruster_3">
+    <self_collide>false</self_collide>
+    <inertial>
+      <mass value="0.001"/>
+      <origin xyz="0.12 -0.12 0.2" rpy="0 -1.5708 0"/>
+      <inertia ixx="0.00001" ixy="0.0" ixz="0.0" iyy="0.00001" iyz="0.0" izz="0.00001"/>
+    </inertial>
+  </link>
+  <joint name='${prefix}thruster_3_joint' type='fixed'>
+    <parent link="${prefix}body" />
+    <child link="${prefix}thruster_3" />
+    <use_parent_model_frame>1</use_parent_model_frame>
+  </joint>
+  <gazebo reference="${prefix}thruster_3_joint">
+    <preserveFixedJoint>true</preserveFixedJoint>
+  </gazebo>
+  <link name="${prefix}thruster_4">
+    <self_collide>false</self_collide>
+    <inertial>
+      <mass value="0.001"/>
+      <origin xyz="0.12 0.12 0.2" rpy="1.5708 0 0"/>
+      <inertia ixx="0.00001" ixy="0.0" ixz="0.0" iyy="0.00001" iyz="0.0" izz="0.00001"/>
+    </inertial>
+  </link>
+  <joint name='${prefix}thruster_4_joint' type='fixed'>
+    <parent link="${prefix}body" />
+    <child link="${prefix}thruster_4" />
+    <use_parent_model_frame>1</use_parent_model_frame>
+  </joint>
+  <gazebo reference="${prefix}thruster_4_joint">
+    <preserveFixedJoint>true</preserveFixedJoint>
+  </gazebo>
+  <link name="${prefix}thruster_5">
+    <self_collide>false</self_collide>
+    <inertial>
+      <mass value="0.001"/>
+      <origin xyz="0.12 -0.12 0.2" rpy="-1.5708 0 0"/>
+      <inertia ixx="0.00001" ixy="0.0" ixz="0.0" iyy="0.00001" iyz="0.0" izz="0.00001"/>
+    </inertial>
+  </link>
+  <joint name='${prefix}thruster_5_joint' type='fixed'>
+    <parent link="${prefix}body" />
+    <child link="${prefix}thruster_5" />
+    <use_parent_model_frame>1</use_parent_model_frame>
+  </joint>
+  <gazebo reference="${prefix}thruster_5_joint">
+    <preserveFixedJoint>true</preserveFixedJoint>
+  </gazebo>
+  <link name="${prefix}thruster_6">
+    <self_collide>false</self_collide>
+    <inertial>
+      <mass value="0.001"/>
+      <origin xyz="-0.12 0.12 0.2" rpy="1.5708 0 0"/>
+      <inertia ixx="0.00001" ixy="0.0" ixz="0.0" iyy="0.00001" iyz="0.0" izz="0.00001"/>
+    </inertial>
+  </link>
+  <joint name='${prefix}thruster_6_joint' type='fixed'>
+    <parent link="${prefix}body" />
+    <child link="${prefix}thruster_6" />
+    <use_parent_model_frame>1</use_parent_model_frame>
+  </joint>
+  <gazebo reference="${prefix}thruster_6_joint">
+    <preserveFixedJoint>true</preserveFixedJoint>
+  </gazebo>
+  <link name="${prefix}thruster_7">
+    <self_collide>false</self_collide>
+    <inertial>
+      <mass value="0.001"/>
+      <origin xyz="-0.12 -0.12 0.2" rpy="-1.5708 0 0"/>
+      <inertia ixx="0.00001" ixy="0.0" ixz="0.0" iyy="0.00001" iyz="0.0" izz="0.00001"/>
+    </inertial>
+  </link>
+  <joint name='${prefix}thruster_7_joint' type='fixed'>
+    <parent link="${prefix}body" />
+    <child link="${prefix}thruster_7" />
+    <use_parent_model_frame>1</use_parent_model_frame>
+  </joint>
+  <gazebo reference="${prefix}thruster_7_joint">
+    <preserveFixedJoint>true</preserveFixedJoint>
+  </gazebo>
   <gazebo reference="${prefix}body">
     <kp>100000.0</kp>
@@ -66,8 +189,8 @@
   </gazebo>
   <!-- MODEL-->
-  <xacro:include filename="$(find discower_description)/urdf/model_drag.urdf.xacro" />
-  <xacro:include filename="$(find discower_description)/urdf/model_thrusters.urdf.xacro" />
-  <xacro:include filename="$(find discower_description)/urdf/model_truth.urdf.xacro" />
-  <xacro:include filename="$(find discower_description)/urdf/model_sitl.urdf.xacro" />
+  <xacro:include filename="$(find discower_description)/urdf/model_drag.urdf.xacro"/>
+  <xacro:include filename="$(find discower_description)/urdf/model_thrusters.urdf.xacro"/>
+  <xacro:include filename="$(find discower_description)/urdf/model_truth.urdf.xacro"/>
+  <xacro:include filename="$(find discower_description)/urdf/model_sitl.urdf.xacro"/>
   <!-- SENSORS -->
   <!-- <xacro:include filename="$(find discower_description)/urdf/sensor_imu.urdf.xacro" /> -->

File: discower_description/urdf/model_sitl.urdf.xacro (robot description, xacro)
@@ -1,8 +1,8 @@
 <robot xmlns:xacro="http://www.ros.org/wiki/xacro">
- <gazebo>
-    <plugin name='rotors_gazebo_imu_plugin' filename='libgazebo_imu_plugin.so'>
+  <gazebo>
+    <plugin name='${prefix}rotors_gazebo_imu_plugin' filename='libgazebo_imu_plugin.so'>
       <robotNamespace/>
       <linkName>${prefix}body</linkName>
-      <imuTopic>/imu</imuTopic>
+      <imuTopic>${prefix}/imu</imuTopic>
       <gyroscopeNoiseDensity>0.00018665</gyroscopeNoiseDensity>
       <gyroscopeRandomWalk>3.8785e-05</gyroscopeRandomWalk>
@@ -14,8 +14,8 @@
       <accelerometerTurnOnBiasSigma>0.196</accelerometerTurnOnBiasSigma>
     </plugin>
-    <plugin name='groundtruth_plugin' filename='libgazebo_groundtruth_plugin.so'>
+    <plugin name='${prefix}groundtruth_plugin' filename='libgazebo_groundtruth_plugin.so'>
       <robotNamespace/>
     </plugin>
-    <plugin name='magnetometer_plugin' filename='libgazebo_magnetometer_plugin.so'>
+    <plugin name='${prefix}magnetometer_plugin' filename='libgazebo_magnetometer_plugin.so'>
       <robotNamespace/>
       <pubRate>100</pubRate>
@@ -23,17 +23,17 @@
       <randomWalk>6.4e-06</randomWalk>
       <biasCorrelationTime>600</biasCorrelationTime>
-      <magTopic>/mag</magTopic>
+      <magTopic>${prefix}/mag</magTopic>
     </plugin>
-    <plugin name='barometer_plugin' filename='libgazebo_barometer_plugin.so'>
+    <plugin name='${prefix}barometer_plugin' filename='libgazebo_barometer_plugin.so'>
       <robotNamespace/>
       <pubRate>50</pubRate>
-      <baroTopic>/baro</baroTopic>
+      <baroTopic>${prefix}/baro</baroTopic>
       <baroDriftPaPerSec>0</baroDriftPaPerSec>
     </plugin>
-    <plugin name='mavlink_interface' filename='libgazebo_mavlink_interface.so'>
+    <plugin name='${prefix}mavlink_interface' filename='libgazebo_mavlink_interface.so'>
       <robotNamespace/>
-      <imuSubTopic>/imu</imuSubTopic>
-      <magSubTopic>/mag</magSubTopic>
-      <baroSubTopic>/baro</baroSubTopic>
+      <imuSubTopic>${prefix}/imu</imuSubTopic>
+      <magSubTopic>${prefix}/mag</magSubTopic>
+      <baroSubTopic>${prefix}/baro</baroSubTopic>
       <mavlink_addr>INADDR_ANY</mavlink_addr>
       <mavlink_tcp_port>4560</mavlink_tcp_port>
@@ -52,99 +52,37 @@
       <enable_lockstep>1</enable_lockstep>
       <use_tcp>1</use_tcp>
-      <motorSpeedCommandPubTopic>/gazebo/command/motor_speed</motorSpeedCommandPubTopic>
+      <actuatorOutputsCommandPubTopic>${prefix}/gazebo/command/actuator_outputs</actuatorOutputsCommandPubTopic>
       <control_channels>
-        <channel name='rotor1'>
+        <channel name='thruster1'>
           <input_index>0</input_index>
-          <input_offset>0</input_offset>
-          <input_scaling>1000</input_scaling>
-          <zero_position_disarmed>0</zero_position_disarmed>
-          <zero_position_armed>100</zero_position_armed>
-          <joint_control_type>velocity</joint_control_type>
+          <joint_control_type>bypass</joint_control_type>
         </channel>
-        <channel name='rotor2'>
+        <channel name='thruster2'>
           <input_index>1</input_index>
-          <input_offset>0</input_offset>
-          <input_scaling>1000</input_scaling>
-          <zero_position_disarmed>0</zero_position_disarmed>
-          <zero_position_armed>100</zero_position_armed>
-          <joint_control_type>velocity</joint_control_type>
+          <joint_control_type>bypass</joint_control_type>
         </channel>
-        <channel name='rotor3'>
+        <channel name='thruster3'>
           <input_index>2</input_index>
-          <input_offset>0</input_offset>
-          <input_scaling>1000</input_scaling>
-          <zero_position_disarmed>0</zero_position_disarmed>
-          <zero_position_armed>100</zero_position_armed>
-          <joint_control_type>velocity</joint_control_type>
+          <joint_control_type>bypass</joint_control_type>
         </channel>
-        <channel name='rotor4'>
+        <channel name='thruster4'>
           <input_index>3</input_index>
-          <input_offset>0</input_offset>
-          <input_scaling>1000</input_scaling>
-          <zero_position_disarmed>0</zero_position_disarmed>
-          <zero_position_armed>100</zero_position_armed>
-          <joint_control_type>velocity</joint_control_type>
+          <joint_control_type>bypass</joint_control_type>
         </channel>
-        <channel name='rotor5'>
+        <channel name='thruster5'>
           <input_index>4</input_index>
-          <input_offset>1</input_offset>
-          <input_scaling>324.6</input_scaling>
-          <zero_position_disarmed>0</zero_position_disarmed>
-          <zero_position_armed>0</zero_position_armed>
-          <joint_control_type>velocity</joint_control_type>
-          <joint_control_pid>
-            <p>0.1</p>
-            <i>0</i>
-            <d>0</d>
-            <iMax>0.0</iMax>
-            <iMin>0.0</iMin>
-            <cmdMax>2</cmdMax>
-            <cmdMin>-2</cmdMin>
-          </joint_control_pid>
-          <joint_name>zephyr_delta_wing::propeller_joint</joint_name>
+          <joint_control_type>bypass</joint_control_type>
         </channel>
-        <channel name='rotor6'>
+        <channel name='thruster6'>
           <input_index>5</input_index>
-          <input_offset>0</input_offset>
-          <input_scaling>0.524</input_scaling>
-          <zero_position_disarmed>0</zero_position_disarmed>
-          <zero_position_armed>0</zero_position_armed>
-          <joint_control_type>position</joint_control_type>
-          <joint_name>zephyr_delta_wing::flap_left_joint</joint_name>
-          <joint_control_pid>
-            <p>10.0</p>
-            <i>0</i>
-            <d>0</d>
-            <iMax>0</iMax>
-            <iMin>0</iMin>
-            <cmdMax>20</cmdMax>
-            <cmdMin>-20</cmdMin>
-          </joint_control_pid>
+          <joint_control_type>bypass</joint_control_type>
         </channel>
-        <channel name='rotor7'>
+        <channel name='thruster7'>
           <input_index>6</input_index>
-          <input_offset>0</input_offset>
-          <input_scaling>0.524</input_scaling>
-          <zero_position_disarmed>0</zero_position_disarmed>
-          <zero_position_armed>0</zero_position_armed>
-          <joint_control_type>position</joint_control_type>
-          <joint_name>zephyr_delta_wing::flap_right_joint</joint_name>
-          <joint_control_pid>
-            <p>10.0</p>
-            <i>0</i>
-            <d>0</d>
-            <iMax>0</iMax>
-            <iMin>0</iMin>
-            <cmdMax>20</cmdMax>
-            <cmdMin>-20</cmdMin>
-          </joint_control_pid>
+          <joint_control_type>bypass</joint_control_type>
         </channel>
-        <channel name='rotor8'>
+        <channel name='thruster8'>
           <input_index>7</input_index>
-          <input_offset>0</input_offset>
-          <input_scaling>0.524</input_scaling>
-          <zero_position_disarmed>0</zero_position_disarmed>
-          <zero_position_armed>0</zero_position_armed>
-          <joint_control_type>position</joint_control_type>
+          <joint_control_type>bypass</joint_control_type>
         </channel>
       </control_channels>

File: discower_description/urdf/model_thrusters.urdf.xacro (robot description, xacro)
@@ -1,24 +1,68 @@
 <?xml version="1.0"?>
-<!-- Copyright (c) 2017, United States Government, as represented by the     -->
-<!-- Administrator of the National Aeronautics and Space Administration.     -->
-<!--                                                                         -->
-<!-- All rights reserved.                                                    -->
-<!--                                                                         -->
-<!-- The Astrobee platform is licensed under the Apache License, Version 2.0 -->
-<!-- (the "License"); you may not use this file except in compliance with    -->
-<!-- the License. You may obtain a copy of the License at                    -->
-<!--                                                                         -->
-<!--     http://www.apache.org/licenses/LICENSE-2.0                          -->
-<!--                                                                         -->
-<!-- Unless required by applicable law or agreed to in writing, software     -->
-<!-- distributed under the License is distributed on an "AS IS" BASIS,       -->
-<!-- WITHOUT WARRANTIES OR CONDITIONS OF ANY KIND, either express or         -->
-<!-- implied. See the License for the specific language governing            -->
-<!-- permissions and limitations under the License.                          -->
 <robot xmlns:xacro="http://www.ros.org/wiki/xacro">
   <gazebo>
-    <plugin name="thrusters_ros" filename="libgazebo_model_plugin_thrusters.so">
-      <rate>10.0</rate>
-      <bypass_thrusters_model>true</bypass_thrusters_model>
+    <plugin name='thruster_0_model' filename='libgazebo_coldgas_thruster_plugin.so'>
+      <robotNamespace/>
+      <linkName>${prefix}thruster_0</linkName>
+      <thrusterNumber>0</thrusterNumber>
+      <commandSubTopic>${prefix}/gazebo/command/actuator_outputs</commandSubTopic>
+      <pwmFrequency>10</pwmFrequency>
+      <maxThrust>1.4</maxThrust>
+    </plugin>
+    <plugin name='thruster_1_model' filename='libgazebo_coldgas_thruster_plugin.so'>
+      <robotNamespace/>
+      <linkName>${prefix}thruster_1</linkName>
+      <thrusterNumber>1</thrusterNumber>
+      <commandSubTopic>${prefix}/gazebo/command/actuator_outputs</commandSubTopic>
+      <pwmFrequency>10</pwmFrequency>
+      <maxThrust>1.4</maxThrust>
+    </plugin>
+    <plugin name='thruster_2_model' filename='libgazebo_coldgas_thruster_plugin.so'>
+      <robotNamespace/>
+      <linkName>${prefix}thruster_2</linkName>
+      <thrusterNumber>2</thrusterNumber>
+      <commandSubTopic>${prefix}/gazebo/command/actuator_outputs</commandSubTopic>
+      <pwmFrequency>10</pwmFrequency>
+      <maxThrust>1.4</maxThrust>
+    </plugin>
+    <plugin name='thruster_3_model' filename='libgazebo_coldgas_thruster_plugin.so'>
+      <robotNamespace/>
+      <linkName>${prefix}thruster_3</linkName>
+      <thrusterNumber>3</thrusterNumber>
+      <commandSubTopic>${prefix}/gazebo/command/actuator_outputs</commandSubTopic>
+      <pwmFrequency>10</pwmFrequency>
+      <maxThrust>1.4</maxThrust>
+    </plugin>
+    <plugin name='thruster_4_model' filename='libgazebo_coldgas_thruster_plugin.so'>
+      <robotNamespace/>
+      <linkName>${prefix}thruster_4</linkName>
+      <thrusterNumber>4</thrusterNumber>
+      <commandSubTopic>${prefix}/gazebo/command/actuator_outputs</commandSubTopic>
+      <pwmFrequency>10</pwmFrequency>
+      <maxThrust>1.4</maxThrust>
+    </plugin>
+    <plugin name='thruster_5_model' filename='libgazebo_coldgas_thruster_plugin.so'>
+      <robotNamespace/>
+      <linkName>${prefix}thruster_5</linkName>
+      <thrusterNumber>5</thrusterNumber>
+      <commandSubTopic>${prefix}/gazebo/command/actuator_outputs</commandSubTopic>
+      <pwmFrequency>10</pwmFrequency>
+      <maxThrust>1.4</maxThrust>
+    </plugin>
+    <plugin name='thruster_6_model' filename='libgazebo_coldgas_thruster_plugin.so'>
+      <robotNamespace/>
+      <linkName>${prefix}thruster_6</linkName>
+      <thrusterNumber>6</thrusterNumber>
+      <commandSubTopic>${prefix}/gazebo/command/actuator_outputs</commandSubTopic>
+      <pwmFrequency>10</pwmFrequency>
+      <maxThrust>1.4</maxThrust>
+    </plugin>
+    <plugin name='thruster_7_model' filename='libgazebo_coldgas_thruster_plugin.so'>
+      <robotNamespace/>
+      <linkName>${prefix}thruster_7</linkName>
+      <thrusterNumber>7</thrusterNumber>
+      <commandSubTopic>${prefix}/gazebo/command/actuator_outputs</commandSubTopic>
+      <pwmFrequency>10</pwmFrequency>
+      <maxThrust>1.4</maxThrust>
     </plugin>
   </gazebo>

File: discower_description/urdf/model_thrusters_gz.urdf.xacro (robot description, xacro)
@@ -18,12 +18,7 @@
 <robot xmlns:xacro="http://www.ros.org/wiki/xacro">
   <gazebo>
-    <plugin name="truth_ros" filename="libgazebo_model_plugin_truth.so">
-      <rate>62.5</rate>
-      <parent>world</parent>
-      <child>${prefix}truth</child>
-      <tf>true</tf>
-      <pose>true</pose>
-      <twist>true</twist>
-      <static>false</static>
+    <plugin name="thrusters_ros" filename="libgazebo_model_plugin_thrusters.so">
+      <rate>10.0</rate>
+      <bypass_thrusters_model>true</bypass_thrusters_model>
     </plugin>
   </gazebo>
