Commit message: fix: joint locations

File: discower_description/urdf/model.urdf.xacro (robot description, xacro)
@@ -57,5 +57,5 @@
     <inertial>
       <mass value="0.001"/>
-      <origin xyz="-0.12 0.12 0.2" rpy="0 1.5708 0"/>
+      <origin xyz="0 0 0" rpy="0 0 0"/>
       <inertia ixx="0.00001" ixy="0.0" ixz="0.0" iyy="0.00001" iyz="0.0" izz="0.00001"/>
     </inertial>
@@ -64,4 +64,5 @@
     <parent link="${prefix}body" />
     <child link="${prefix}thruster_0" />
+    <origin xyz="-0.12 0.12 0.2" rpy="0 1.5708 0"/>
     <use_parent_model_frame>1</use_parent_model_frame>
   </joint>
@@ -73,5 +74,5 @@
     <inertial>
       <mass value="0.001"/>
-      <origin xyz="0.12 0.12 0.2" rpy="0 -1.5708 0"/>
+      <origin xyz="0 0 0" rpy="0 0 0"/>
       <inertia ixx="0.00001" ixy="0.0" ixz="0.0" iyy="0.00001" iyz="0.0" izz="0.00001"/>
     </inertial>
@@ -80,4 +81,5 @@
     <parent link="${prefix}body" />
     <child link="${prefix}thruster_1" />
+    <origin xyz="0.12 0.12 0.2" rpy="0 -1.5708 0"/>
     <use_parent_model_frame>1</use_parent_model_frame>
   </joint>
@@ -89,5 +91,5 @@
     <inertial>
       <mass value="0.001"/>
-      <origin xyz="-0.12 -0.12 0.2" rpy="0 1.5708 0"/>
+      <origin xyz="0 0 0" rpy="0 0 0"/>
       <inertia ixx="0.00001" ixy="0.0" ixz="0.0" iyy="0.00001" iyz="0.0" izz="0.00001"/>
     </inertial>
@@ -96,4 +98,5 @@
     <parent link="${prefix}body" />
     <child link="${prefix}thruster_2" />
+    <origin xyz="-0.12 -0.12 0.2" rpy="0 1.5708 0"/>
     <use_parent_model_frame>1</use_parent_model_frame>
   </joint>
@@ -105,5 +108,5 @@
     <inertial>
       <mass value="0.001"/>
-      <origin xyz="0.12 -0.12 0.2" rpy="0 -1.5708 0"/>
+      <origin xyz="0 0 0" rpy="0 0 0"/>
       <inertia ixx="0.00001" ixy="0.0" ixz="0.0" iyy="0.00001" iyz="0.0" izz="0.00001"/>
     </inertial>
@@ -112,4 +115,5 @@
     <parent link="${prefix}body" />
     <child link="${prefix}thruster_3" />
+    <origin xyz="0.12 -0.12 0.2" rpy="0 -1.5708 0"/>
     <use_parent_model_frame>1</use_parent_model_frame>
   </joint>
@@ -121,5 +125,5 @@
     <inertial>
       <mass value="0.001"/>
-      <origin xyz="0.12 0.12 0.2" rpy="1.5708 0 0"/>
+      <origin xyz="0 0 0" rpy="0 0 0"/>
       <inertia ixx="0.00001" ixy="0.0" ixz="0.0" iyy="0.00001" iyz="0.0" izz="0.00001"/>
     </inertial>
@@ -128,4 +132,5 @@
     <parent link="${prefix}body" />
     <child link="${prefix}thruster_4" />
+    <origin xyz="0.12 0.12 0.2" rpy="1.5708 0 0"/>
     <use_parent_model_frame>1</use_parent_model_frame>
   </joint>
@@ -137,5 +142,5 @@
     <inertial>
       <mass value="0.001"/>
-      <origin xyz="0.12 -0.12 0.2" rpy="-1.5708 0 0"/>
+      <origin xyz="0 0 0" rpy="0 0 0"/>
       <inertia ixx="0.00001" ixy="0.0" ixz="0.0" iyy="0.00001" iyz="0.0" izz="0.00001"/>
     </inertial>
@@ -144,4 +149,5 @@
     <parent link="${prefix}body" />
     <child link="${prefix}thruster_5" />
+    <origin xyz="0.12 -0.12 0.2" rpy="-1.5708 0 0"/>
     <use_parent_model_frame>1</use_parent_model_frame>
   </joint>
@@ -153,5 +159,5 @@
     <inertial>
       <mass value="0.001"/>
-      <origin xyz="-0.12 0.12 0.2" rpy="1.5708 0 0"/>
+      <origin xyz="0 0 0" rpy="0 0 0"/>
       <inertia ixx="0.00001" ixy="0.0" ixz="0.0" iyy="0.00001" iyz="0.0" izz="0.00001"/>
     </inertial>
@@ -160,4 +166,5 @@
     <parent link="${prefix}body" />
     <child link="${prefix}thruster_6" />
+    <origin xyz="-0.12 0.12 0.2" rpy="1.5708 0 0"/>
     <use_parent_model_frame>1</use_parent_model_frame>
   </joint>
@@ -169,5 +176,5 @@
     <inertial>
       <mass value="0.001"/>
-      <origin xyz="-0.12 -0.12 0.2" rpy="-1.5708 0 0"/>
+      <origin xyz="0 0 0" rpy="0 0 0"/>
       <inertia ixx="0.00001" ixy="0.0" ixz="0.0" iyy="0.00001" iyz="0.0" izz="0.00001"/>
     </inertial>
@@ -176,4 +183,5 @@
     <parent link="${prefix}body" />
     <child link="${prefix}thruster_7" />
+    <origin xyz="-0.12 -0.12 0.2" rpy="-1.5708 0 0"/>
     <use_parent_model_frame>1</use_parent_model_frame>
   </joint>
